File: Lab8 Schematic/Lab8 Schematic.kicad_pcb (KiCad board)
At the start: 2 copper layers, 85 x 39 mm, 13 parts, among them U4 ACPL-214-500E

Commit message: All signoffs received
Parts:
- C1, C2: footprint Capacitor_SMD:C_0201_0603Metric -> Capacitor_THT:CP_Axial_L10.0mm_D4.5mm_P15.00mm_Horizontal
- R1, R2, R3, R4, R5: footprint Resistor_SMD:R_0201_0603Metric -> Resistor_THT:R_Axial_DIN0207_L6.3mm_D2.5mm_P2.54mm_Vertical
- moved C2 9.24 mm to (149.5, 56.3)
- moved R1 8.80 mm to (116.0, 65.5)
- moved C1 7.00 mm to (111.0, 56.7)
- moved R3 6.34 mm to (142.5, 65.5)
Routing:
- net GND: track 43.0 -> 56.5 mm
- net Net-(R4-Pad2): track 32.1 -> 39.6 mm
- net Net-(U3-+): track 23.4 -> 20.4 mm
- net Net-(D1-A): track 18.2 -> 16.0 mm
- net Net-(U2-+): track 20.4 -> 22.4 mm
- net Net-(U3--): track 34.4 -> 36.2 mm
- net Net-(U1--): track 20.1 -> 20.8 mm
- net Net-(U2--): track 44.1 -> 44.6 mm
Other:
- board size 85 x 39 mm -> 81.5 x 41.5 mm
