File: Lab8 Schematic/Lab8 Schematic.kicad_sch (KiCad schematic)
At the start: 13 parts, among them U1 ${SIM.PARAMS}, U2 ${SIM.PARAMS}, U3 ${SIM.PARAMS}

Commit message: KiCad schematic done, PCB has a strange error
Parts:
- removed BT1, BT2: Battery_Cell, symbol Device:Battery_Cell
- removed D1: D_Schottky_Dual_Series_KCA_Split, symbol Device:D_Schottky_Dual_Series_KCA_Split
- added D1, D2: 1N5819, Diode_THT:D_DO-41_SOD81_P10.16mm_Horizontal, symbol Diode:1N5819
- added U4: ACPL-214-500E, Package_SO:SOP-4_4.4x2.6mm_P1.27mm, symbol Isolator:ACPL-214-500E
- C1: value C -> 19u; footprint (none) -> Capacitor_SMD:C_0201_0603Metric
- C2: value C -> 4u; footprint (none) -> Capacitor_SMD:C_0201_0603Metric
- R1, R2: value R_US -> 10k; footprint (none) -> Resistor_SMD:R_0201_0603Metric
- R3: value R_US -> 1k; footprint (none) -> Resistor_SMD:R_0201_0603Metric
- R4: value R_US -> 28k; footprint (none) -> Resistor_SMD:R_0201_0603Metric
- R5: value R_US -> 100; footprint (none) -> Resistor_SMD:R_0201_0603Metric
- U1, U2, U3: footprint (none) -> Package_DIP:DIP-8_W7.62mm_SMDSocket_SmallPads
Connections:
- net +5V: now also U4.1
- net -3V3: now also D2.2 (A)
- net GND: now also U4.2, U4.3
- net at R5.2: now also D1.2 (A), D2.1 (K)
- net at U1.1 (+): now also U4.4
- new net +3.3V: D1.1 (K)

Commit message: All signoffs received
Parts:
- C1, C2: footprint Capacitor_SMD:C_0201_0603Metric -> Capacitor_THT:CP_Axial_L10.0mm_D4.5mm_P15.00mm_Horizontal
- R1, R2, R3, R4, R5: footprint Resistor_SMD:R_0201_0603Metric -> Resistor_THT:R_Axial_DIN0207_L6.3mm_D2.5mm_P2.54mm_Vertical
Changed lines of the file:
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@@
 			)
 		)
-		(property "Footprint" "Resistor_SMD:R_0201_0603Metric"
+		(property "Footprint" "Resistor_THT:R_Axial_DIN0207_L6.3mm_D2.5mm_P2.54mm_Vertical"
 			(at 145.034 95.504 90)
 			(effects
@@
 			)
 		)
-		(property "Footprint" "Resistor_SMD:R_0201_0603Metric"
+		(property "Footprint" "Resistor_THT:R_Axial_DIN0207_L6.3mm_D2.5mm_P2.54mm_Vertical"
 			(at 164.846 119.634 90)
 			(effects
@@
 			)
 		)
-		(property "Footprint" "Capacitor_SMD:C_0201_0603Metric"
+		(property "Footprint" "Capacitor_THT:CP_Axial_L10.0mm_D4.5mm_P15.00mm_Horizontal"
 			(at 153.3652 111.76 0)
 			(effects
@@
 			)
 		)
-		(property "Footprint" "Resistor_SMD:R_0201_0603Metric"
+		(property "Footprint" "Resistor_THT:R_Axial_DIN0207_L6.3mm_D2.5mm_P2.54mm_Vertical"
 			(at 195.834 114.554 90)
 			(effects
@@
 			)
 		)
-		(property "Footprint" "Resistor_SMD:R_0201_0603Metric"
+		(property "Footprint" "Resistor_THT:R_Axial_DIN0207_L6.3mm_D2.5mm_P2.54mm_Vertical"
 			(at 180.594 114.554 90)
 			(effects
@@
 			)
 		)
-		(property "Footprint" "Resistor_SMD:R_0201_0603Metric"
+		(property "Footprint" "Resistor_THT:R_Axial_DIN0207_L6.3mm_D2.5mm_P2.54mm_Vertical"
 			(at 115.316 109.474 90)
 			(effects
@@
 			)
 		)
-		(property "Footprint" "Capacitor_SMD:C_0201_0603Metric"
+		(property "Footprint" "Capacitor_THT:CP_Axial_L10.0mm_D4.5mm_P15.00mm_Horizontal"
 			(at 111.76 93.0148 0)
 			(effects
